Commit message: Added use_docking_adapter condition in srdf

File: neo_ur_moveit_config/srdf/mpo_700.srdf.xacro (robot description, xacro)
@@ -7,4 +7,5 @@
      <xacro:arg name="prefix" default=""/>
      <xacro:property name="prefix_value" value="$(arg prefix)"/>
+     <xacro:arg name="use_docking_adapter" default="false"/>
     <!--GROUPS: Representation of a set of joints and links. This can be useful for specifying DOF to plan for, defining arms, end effectors, etc-->
     <!--LINKS: When a link is specified, the parent joint of that link (if it exists) is automatically included-->
@@ -23,18 +24,18 @@
     <!--GROUP STATES: Purpose: Define a named state for a particular group, in terms of joint values. This is useful to define states like 'folded arms'-->
     <group_state name="up" group="ur_manipulator">
-      <joint name="${prefix_value}elbow_joint" value="0" />
-      <joint name="${prefix_value}shoulder_lift_joint" value="-1.5707" />
-      <joint name="${prefix_value}shoulder_pan_joint" value="0" />
-      <joint name="${prefix_value}wrist_1_joint" value="-1.5707" />
-      <joint name="${prefix_value}wrist_2_joint" value="0" />
-      <joint name="${prefix_value}wrist_3_joint" value="0" />
+        <joint name="${prefix_value}elbow_joint" value="0" />
+        <joint name="${prefix_value}shoulder_lift_joint" value="-1.5707" />
+        <joint name="${prefix_value}shoulder_pan_joint" value="0" />
+        <joint name="${prefix_value}wrist_1_joint" value="-1.5707" />
+        <joint name="${prefix_value}wrist_2_joint" value="0" />
+        <joint name="${prefix_value}wrist_3_joint" value="0" />
     </group_state>
     <group_state name="test_configuration" group="ur_manipulator">
-      <joint name="${prefix_value}elbow_joint" value="1.4" />
-      <joint name="${prefix_value}shoulder_lift_joint" value="-1.62" />
-      <joint name="${prefix_value}shoulder_pan_joint" value="1.54" />
-      <joint name="${prefix_value}wrist_1_joint" value="-1.2" />
-      <joint name="${prefix_value}wrist_2_joint" value="-1.6" />
-      <joint name="${prefix_value}wrist_3_joint" value="-0.11" />
+        <joint name="${prefix_value}elbow_joint" value="1.4" />
+        <joint name="${prefix_value}shoulder_lift_joint" value="-1.62" />
+        <joint name="${prefix_value}shoulder_pan_joint" value="1.54" />
+        <joint name="${prefix_value}wrist_1_joint" value="-1.2" />
+        <joint name="${prefix_value}wrist_2_joint" value="-1.6" />
+        <joint name="${prefix_value}wrist_3_joint" value="-0.11" />
     </group_state>
     <!--DISABLE COLLISIONS: By default it is assumed that any link of the robot could potentially come into collision with any other link in the robot. This tag disables collision checking between a specified pair of links. -->
@@ -66,17 +67,20 @@
     <disable_collisions link1="cabinet_link" link2="${prefix_value}base_link_inertia" reason="Adjacent"/>
     <disable_collisions link1="cabinet_link" link2="${prefix_value}shoulder_link" reason="Never"/>
-    <disable_collisions link1="docking_adapter_link" link2="lidar_1_link" reason="Never"/>
-    <disable_collisions link1="docking_adapter_link" link2="lidar_2_link" reason="Never"/>
-    <disable_collisions link1="docking_adapter_link" link2="mpo_700_caster_back_left_link" reason="Never"/>
-    <disable_collisions link1="docking_adapter_link" link2="mpo_700_caster_back_right_link" reason="Never"/>
-    <disable_collisions link1="docking_adapter_link" link2="mpo_700_caster_front_left_link" reason="Never"/>
-    <disable_collisions link1="docking_adapter_link" link2="mpo_700_caster_front_right_link" reason="Never"/>
-    <disable_collisions link1="docking_adapter_link" link2="mpo_700_wheel_back_left_link" reason="Never"/>
-    <disable_collisions link1="docking_adapter_link" link2="mpo_700_wheel_back_right_link" reason="Never"/>
-    <disable_collisions link1="docking_adapter_link" link2="mpo_700_wheel_front_left_link" reason="Never"/>
-    <disable_collisions link1="docking_adapter_link" link2="mpo_700_wheel_front_right_link" reason="Never"/>
-    <disable_collisions link1="docking_adapter_link" link2="ur10base_link_inertia" reason="Never"/>
-    <disable_collisions link1="docking_adapter_link" link2="ur10shoulder_link" reason="Never"/>
-    <disable_collisions link1="docking_adapter_link" link2="ur10upper_arm_link" reason="Never"/>
+    <!--Use docking adapter-->
+    <xacro:if value="$(arg use_docking_adapter)">
+        <disable_collisions link1="docking_adapter_link" link2="lidar_1_link" reason="Never"/>
+        <disable_collisions link1="docking_adapter_link" link2="lidar_2_link" reason="Never"/>
+        <disable_collisions link1="docking_adapter_link" link2="mpo_700_caster_back_left_link" reason="Never"/>
+        <disable_collisions link1="docking_adapter_link" link2="mpo_700_caster_back_right_link" reason="Never"/>
+        <disable_collisions link1="docking_adapter_link" link2="mpo_700_caster_front_left_link" reason="Never"/>
+        <disable_collisions link1="docking_adapter_link" link2="mpo_700_caster_front_right_link" reason="Never"/>
+        <disable_collisions link1="docking_adapter_link" link2="mpo_700_wheel_back_left_link" reason="Never"/>
+        <disable_collisions link1="docking_adapter_link" link2="mpo_700_wheel_back_right_link" reason="Never"/>
+        <disable_collisions link1="docking_adapter_link" link2="mpo_700_wheel_front_left_link" reason="Never"/>
+        <disable_collisions link1="docking_adapter_link" link2="mpo_700_wheel_front_right_link" reason="Never"/>
+        <disable_collisions link1="docking_adapter_link" link2="ur10base_link_inertia" reason="Never"/>
+        <disable_collisions link1="docking_adapter_link" link2="ur10shoulder_link" reason="Never"/>
+        <disable_collisions link1="docking_adapter_link" link2="ur10upper_arm_link" reason="Never"/>
+    </xacro:if>
     <disable_collisions link1="lidar_1_link" link2="lidar_2_link" reason="Adjacent"/>
     <disable_collisions link1="lidar_1_link" link2="mpo_700_caster_back_left_link" reason="Never"/>

Commit message: updating gripper xacro macro

File: neo_ur_moveit_config/srdf/mpo_700.srdf.xacro (robot description, xacro)
@@ -5,6 +5,8 @@
 -->
 <robot xmlns:xacro="http://www.ros.org/wiki/xacro" name="mpo_700">
-     <xacro:arg name="prefix" default=""/>
-     <xacro:property name="prefix_value" value="$(arg prefix)"/>
+    <xacro:arg name="prefix" default=""/>
+    <xacro:arg name="gripper_type" default=""/>
+    <xacro:property name="prefix_value" value="$(arg prefix)"/>
+    <xacro:property name="gripper" value="$(arg gripper_type)"/>
     <!--GROUPS: Representation of a set of joints and links. This can be useful for specifying DOF to plan for, defining arms, end effectors, etc-->
     <!--LINKS: When a link is specified, the parent joint of that link (if it exists) is automatically included-->
@@ -13,11 +15,10 @@
     <!--SUBGROUPS: Groups can also be formed by referencing to already defined group names-->
     <group name="ur_manipulator">
-        <joint name="${prefix_value}wrist_1_joint"/>
-        <joint name="${prefix_value}wrist_2_joint"/>
-        <joint name="${prefix_value}wrist_3_joint"/>
-        <joint name="${prefix_value}shoulder_pan_joint"/>
-        <joint name="${prefix_value}shoulder_lift_joint"/>
-        <joint name="${prefix_value}elbow_joint"/>
-        <chain base_link="${prefix_value}base_link" tip_link="${prefix_value}tool0"/>
+      <joint name="${prefix_value}wrist_1_joint"/>
+      <joint name="${prefix_value}wrist_2_joint"/>
+      <joint name="${prefix_value}wrist_3_joint"/>
+      <joint name="${prefix_value}shoulder_pan_joint"/>
+      <joint name="${prefix_value}shoulder_lift_joint"/>
+      <joint name="${prefix_value}elbow_joint"/>
     </group>
     <!--GROUP STATES: Purpose: Define a named state for a particular group, in terms of joint values. This is useful to define states like 'folded arms'-->
@@ -137,16 +138,15 @@
     <disable_collisions link1="mpo_700_wheel_front_right_link" link2="${prefix_value}upper_arm_link" reason="Never"/>
     <disable_collisions link1="${prefix_value}base_link_inertia" link2="${prefix_value}shoulder_link" reason="Adjacent"/>
-    <disable_collisions link1="${prefix_value}base_link_inertia" link2="${prefix_value}upper_arm_link" reason="Never"/>
-    <disable_collisions link1="${prefix_value}base_link_inertia" link2="${prefix_value}wrist_1_link" reason="Never"/>
     <disable_collisions link1="${prefix_value}forearm_link" link2="${prefix_value}upper_arm_link" reason="Adjacent"/>
     <disable_collisions link1="${prefix_value}forearm_link" link2="${prefix_value}wrist_1_link" reason="Adjacent"/>
+    <disable_collisions link1="${prefix_value}forearm_link" link2="${prefix_value}wrist_2_link" reason="Never"/>
     <disable_collisions link1="${prefix_value}shoulder_link" link2="${prefix_value}upper_arm_link" reason="Adjacent"/>
-    <disable_collisions link1="${prefix_value}shoulder_link" link2="${prefix_value}wrist_1_link" reason="Never"/>
-    <disable_collisions link1="${prefix_value}shoulder_link" link2="${prefix_value}wrist_2_link" reason="Never"/>
     <disable_collisions link1="${prefix_value}wrist_1_link" link2="${prefix_value}wrist_2_link" reason="Adjacent"/>
     <disable_collisions link1="${prefix_value}wrist_1_link" link2="${prefix_value}wrist_3_link" reason="Never"/>
     <disable_collisions link1="${prefix_value}wrist_2_link" link2="${prefix_value}wrist_3_link" reason="Adjacent"/>
-    <disable_collisions link1="${prefix_value}tool0" link2="${prefix_value}wrist_1_link" reason="Never" />
-    <disable_collisions link1="${prefix_value}tool0" link2="${prefix_value}wrist_2_link" reason="Never" />
-    <disable_collisions link1="${prefix_value}tool0" link2="${prefix_value}wrist_3_link" reason="Adjacent" />
+    <!-- Assigning Xacro properties -->
+    <xacro:unless value="${gripper == ''}">
+      <xacro:include filename="$(find neo_ur_moveit_config)/srdf/robotiq_2f_140.xacro" />
+      <xacro:robotiq_2f_140 />
+    </xacro:unless>
 </robot>

Commit message: Gripper addition (#10)
* Functionality/mpo 500 support (#6)

* Added launch argument to change neo robot; generated and included mpo500 srdf for moveit

* Refined launch file code, added joint limits param, changed package structure, tested with neo_simulation2 pkg for mpo_500 and mpo_700 robots with both ur10 and ur5e arm moveit support

* Updated README.md

* Added dynamic parameter substitution for ur controller and joint_limits files

* Updated robot base options

* Removed redundant joint_limit files and Updated README

* updating planning_scene_monitor_parameters

* updating gripper xacro macro

* adding epick support

---------

Co-authored-by: Adarsh Karan Kesavadas Prasanth <112091438+AdarshKaran@users.noreply.github.com>

File: neo_ur_moveit_config/srdf/mpo_700.srdf.xacro (robot description, xacro)
@@ -5,6 +5,8 @@
 -->
 <robot xmlns:xacro="http://www.ros.org/wiki/xacro" name="mpo_700">
-     <xacro:arg name="prefix" default=""/>
-     <xacro:property name="prefix_value" value="$(arg prefix)"/>
+    <xacro:arg name="prefix" default=""/>
+    <xacro:arg name="gripper_type" default=""/>
+    <xacro:property name="prefix_value" value="$(arg prefix)"/>
+    <xacro:property name="gripper" value="$(arg gripper_type)"/>
     <!--GROUPS: Representation of a set of joints and links. This can be useful for specifying DOF to plan for, defining arms, end effectors, etc-->
     <!--LINKS: When a link is specified, the parent joint of that link (if it exists) is automatically included-->
@@ -13,11 +15,10 @@
     <!--SUBGROUPS: Groups can also be formed by referencing to already defined group names-->
     <group name="ur_manipulator">
-        <joint name="${prefix_value}wrist_1_joint"/>
-        <joint name="${prefix_value}wrist_2_joint"/>
-        <joint name="${prefix_value}wrist_3_joint"/>
-        <joint name="${prefix_value}shoulder_pan_joint"/>
-        <joint name="${prefix_value}shoulder_lift_joint"/>
-        <joint name="${prefix_value}elbow_joint"/>
-        <chain base_link="${prefix_value}base_link" tip_link="${prefix_value}tool0"/>
+      <joint name="${prefix_value}wrist_1_joint"/>
+      <joint name="${prefix_value}wrist_2_joint"/>
+      <joint name="${prefix_value}wrist_3_joint"/>
+      <joint name="${prefix_value}shoulder_pan_joint"/>
+      <joint name="${prefix_value}shoulder_lift_joint"/>
+      <joint name="${prefix_value}elbow_joint"/>
     </group>
     <!--GROUP STATES: Purpose: Define a named state for a particular group, in terms of joint values. This is useful to define states like 'folded arms'-->
@@ -137,16 +138,21 @@
     <disable_collisions link1="mpo_700_wheel_front_right_link" link2="${prefix_value}upper_arm_link" reason="Never"/>
     <disable_collisions link1="${prefix_value}base_link_inertia" link2="${prefix_value}shoulder_link" reason="Adjacent"/>
-    <disable_collisions link1="${prefix_value}base_link_inertia" link2="${prefix_value}upper_arm_link" reason="Never"/>
-    <disable_collisions link1="${prefix_value}base_link_inertia" link2="${prefix_value}wrist_1_link" reason="Never"/>
     <disable_collisions link1="${prefix_value}forearm_link" link2="${prefix_value}upper_arm_link" reason="Adjacent"/>
     <disable_collisions link1="${prefix_value}forearm_link" link2="${prefix_value}wrist_1_link" reason="Adjacent"/>
+    <disable_collisions link1="${prefix_value}forearm_link" link2="${prefix_value}wrist_2_link" reason="Never"/>
     <disable_collisions link1="${prefix_value}shoulder_link" link2="${prefix_value}upper_arm_link" reason="Adjacent"/>
-    <disable_collisions link1="${prefix_value}shoulder_link" link2="${prefix_value}wrist_1_link" reason="Never"/>
-    <disable_collisions link1="${prefix_value}shoulder_link" link2="${prefix_value}wrist_2_link" reason="Never"/>
     <disable_collisions link1="${prefix_value}wrist_1_link" link2="${prefix_value}wrist_2_link" reason="Adjacent"/>
     <disable_collisions link1="${prefix_value}wrist_1_link" link2="${prefix_value}wrist_3_link" reason="Never"/>
     <disable_collisions link1="${prefix_value}wrist_2_link" link2="${prefix_value}wrist_3_link" reason="Adjacent"/>
-    <disable_collisions link1="${prefix_value}tool0" link2="${prefix_value}wrist_1_link" reason="Never" />
-    <disable_collisions link1="${prefix_value}tool0" link2="${prefix_value}wrist_2_link" reason="Never" />
-    <disable_collisions link1="${prefix_value}tool0" link2="${prefix_value}wrist_3_link" reason="Adjacent" />
+    <!-- Assigning Xacro properties -->
+    <xacro:unless value="${gripper == ''}">
+      <xacro:if value="${gripper == '2f_140'}">
+        <xacro:include filename="$(find neo_ur_moveit_config)/srdf/robotiq_2f_140.xacro" />
+        <xacro:robotiq_2f_140 />
+      </xacro:if>
+      <xacro:if value="${gripper == 'epick'}">
+        <xacro:include filename="$(find neo_ur_moveit_config)/srdf/robotiq_epick.xacro" />
+        <xacro:robotiq_epick />
+      </xacro:if>
+    </xacro:unless>
 </robot>

Commit message: Removed gripper support completely for moveit, Added 2f_85 gripper support

File: neo_ur_moveit_config/srdf/mpo_700.srdf.xacro (robot description, xacro)
@@ -151,4 +151,8 @@
         <xacro:robotiq_2f_140 />
       </xacro:if>
+      <xacro:if value="${gripper == '2f_85'}">
+        <xacro:include filename="$(find neo_ur_moveit_config)/srdf/robotiq_2f_85.srdf.xacro" />
+        <xacro:robotiq_2f_85 />
+      </xacro:if>
       <xacro:if value="${gripper == 'epick'}">
         <xacro:include filename="$(find neo_ur_moveit_config)/srdf/robotiq_epick.xacro" />

File: neo_ur_moveit_config/srdf/robotiq_2f_140.srdf.xacro (robot description, xacro)
@@ -5,21 +5,8 @@
 -->
 <robot xmlns:xacro="http://www.ros.org/wiki/xacro" name="mpo_700">
+  <xacro:arg name="prefix" default=""/>
+  <xacro:property name="prefix_value" value="$(arg prefix)"/>
   <xacro:macro name="robotiq_2f_140">
-    <!--PASSIVE JOINT: Purpose: this element is used to mark joints that are not actuated-->
-    <!-- <group name="gripper">
-      <joint name="finger_joint"/>
-    </group>
-    <passive_joint name="right_inner_finger_joint"/>
-    <passive_joint name="right_outer_knuckle_joint"/>
-    <passive_joint name="right_inner_knuckle_joint"/>
-    <passive_joint name="left_inner_knuckle_joint"/>
-    <passive_joint name="left_inner_finger_joint"/>
-    <group_state name="open" group="gripper">
-      <joint name="finger_joint" value="0.0" />
-    </group_state>
-    <group_state name="close" group="gripper">
-      <joint name="finger_joint" value="0.695" />
-    </group_state> -->
-    <!-- <end_effector name="endeffector" parent_link="${prefix_value}wrist_3_link" group="gripper"/> -->
+    <!--DISABLE COLLISIONS: By default it is assumed that any link of the robot could potentially come into collision with any other link in the robot. This tag disables collision checking between a specified pair of links. -->
     <disable_collisions link1="left_inner_finger" link2="ur_to_robotiq_link" reason="Never"/>
     <disable_collisions link1="left_inner_finger_pad" link2="ur_to_robotiq_link" reason="Never"/>
