Commit message: Support 2f_140 and 2f_85 robotiq grippers (#12)
* Added gripper 2f_140 robotiq support

* Updating moveit_controllers.yaml for 2f_85 support

* Removed moveit support for gripper

* Removed gripper support completely for moveit, Added 2f_85 gripper support

* Fixed collision issues with mpo_500 srdf and corrected condition logic in launch file

* Updated prefix launch argument description

* Minor formatting and fixes

File: neo_ur_moveit_config/srdf/mpo_500.srdf.xacro (robot description, xacro)
@@ -5,6 +5,8 @@
 -->
 <robot xmlns:xacro="http://www.ros.org/wiki/xacro" name="mpo_500">
-     <xacro:arg name="prefix" default=""/>
-     <xacro:property name="prefix_value" value="$(arg prefix)"/>
+    <xacro:arg name="prefix" default=""/>
+    <xacro:arg name="gripper_type" default=""/>
+    <xacro:property name="prefix_value" value="$(arg prefix)"/>
+    <xacro:property name="gripper" value="$(arg gripper_type)"/>
     <!--GROUPS: Representation of a set of joints and links. This can be useful for specifying DOF to plan for, defining arms, end effectors, etc-->
     <!--LINKS: When a link is specified, the parent joint of that link (if it exists) is automatically included-->
@@ -13,11 +15,11 @@
     <!--SUBGROUPS: Groups can also be formed by referencing to already defined group names-->
     <group name="ur_manipulator">
-        <joint name="${prefix_value}wrist_1_joint"/>
-        <joint name="${prefix_value}wrist_2_joint"/>
-        <joint name="${prefix_value}wrist_3_joint"/>
-        <joint name="${prefix_value}shoulder_pan_joint"/>
-        <joint name="${prefix_value}shoulder_lift_joint"/>
-        <joint name="${prefix_value}elbow_joint"/>
-        <chain base_link="${prefix_value}base_link" tip_link="${prefix_value}tool0"/>
+      <joint name="${prefix_value}wrist_1_joint"/>
+      <joint name="${prefix_value}wrist_2_joint"/>
+      <joint name="${prefix_value}wrist_3_joint"/>
+      <joint name="${prefix_value}shoulder_pan_joint"/>
+      <joint name="${prefix_value}shoulder_lift_joint"/>
+      <joint name="${prefix_value}elbow_joint"/>
+      <chain base_link="${prefix_value}base_link" tip_link="${prefix_value}tool0"/>
     </group>
     <!--GROUP STATES: Purpose: Define a named state for a particular group, in terms of joint values. This is useful to define states like 'folded arms'-->
@@ -42,50 +44,50 @@
     <disable_collisions link1="base_footprint" link2="lidar_1_link" reason="Adjacent"/>
     <disable_collisions link1="base_footprint" link2="lidar_2_link" reason="Adjacent"/>
-    <disable_collisions link1="base_footprint" link2="mpo_500_omni_wheel_back_left_link" reason="Adjacent"/>
-    <disable_collisions link1="base_footprint" link2="mpo_500_omni_wheel_back_right_link" reason="Adjacent"/>
-    <disable_collisions link1="base_footprint" link2="mpo_500_omni_wheel_front_left_link" reason="Adjacent"/>
-    <disable_collisions link1="base_footprint" link2="mpo_500_omni_wheel_front_right_link" reason="Adjacent"/>
+    <disable_collisions link1="base_footprint" link2="mpo_500_wheel_back_left_link" reason="Adjacent"/>
+    <disable_collisions link1="base_footprint" link2="mpo_500_wheel_back_right_link" reason="Adjacent"/>
+    <disable_collisions link1="base_footprint" link2="mpo_500_wheel_front_left_link" reason="Adjacent"/>
+    <disable_collisions link1="base_footprint" link2="mpo_500_wheel_front_right_link" reason="Adjacent"/>
     <disable_collisions link1="base_footprint" link2="${prefix_value}base_link_inertia" reason="Never"/>
     <disable_collisions link1="base_footprint" link2="${prefix_value}shoulder_link" reason="Never"/>
     <disable_collisions link1="cabinet_link" link2="lidar_1_link" reason="Never"/>
     <disable_collisions link1="cabinet_link" link2="lidar_2_link" reason="Never"/>
-    <disable_collisions link1="cabinet_link" link2="mpo_500_omni_wheel_back_left_link" reason="Never"/>
-    <disable_collisions link1="cabinet_link" link2="mpo_500_omni_wheel_back_right_link" reason="Never"/>
-    <disable_collisions link1="cabinet_link" link2="mpo_500_omni_wheel_front_left_link" reason="Never"/>
-    <disable_collisions link1="cabinet_link" link2="mpo_500_omni_wheel_front_right_link" reason="Never"/>
+    <disable_collisions link1="cabinet_link" link2="mpo_500_wheel_back_left_link" reason="Never"/>
+    <disable_collisions link1="cabinet_link" link2="mpo_500_wheel_back_right_link" reason="Never"/>
+    <disable_collisions link1="cabinet_link" link2="mpo_500_wheel_front_left_link" reason="Never"/>
+    <disable_collisions link1="cabinet_link" link2="mpo_500_wheel_front_right_link" reason="Never"/>
     <disable_collisions link1="cabinet_link" link2="${prefix_value}base_link_inertia" reason="Adjacent"/>
     <disable_collisions link1="cabinet_link" link2="${prefix_value}shoulder_link" reason="Never"/>
     <disable_collisions link1="lidar_1_link" link2="lidar_2_link" reason="Never"/>
-    <disable_collisions link1="lidar_1_link" link2="mpo_500_omni_wheel_back_left_link" reason="Never"/>
-    <disable_collisions link1="lidar_1_link" link2="mpo_500_omni_wheel_back_right_link" reason="Never"/>
-    <disable_collisions link1="lidar_1_link" link2="mpo_500_omni_wheel_front_left_link" reason="Never"/>
-    <disable_collisions link1="lidar_1_link" link2="mpo_500_omni_wheel_front_right_link" reason="Never"/>
+    <disable_collisions link1="lidar_1_link" link2="mpo_500_wheel_back_left_link" reason="Never"/>
+    <disable_collisions link1="lidar_1_link" link2="mpo_500_wheel_back_right_link" reason="Never"/>
+    <disable_collisions link1="lidar_1_link" link2="mpo_500_wheel_front_left_link" reason="Never"/>
+    <disable_collisions link1="lidar_1_link" link2="mpo_500_wheel_front_right_link" reason="Never"/>
     <disable_collisions link1="lidar_1_link" link2="${prefix_value}base_link_inertia" reason="Never"/>
     <disable_collisions link1="lidar_1_link" link2="${prefix_value}shoulder_link" reason="Never"/>
-    <disable_collisions link1="lidar_2_link" link2="mpo_500_omni_wheel_back_left_link" reason="Never"/>
-    <disable_collisions link1="lidar_2_link" link2="mpo_500_omni_wheel_back_right_link" reason="Never"/>
-    <disable_collisions link1="lidar_2_link" link2="mpo_500_omni_wheel_front_left_link" reason="Never"/>
-    <disable_collisions link1="lidar_2_link" link2="mpo_500_omni_wheel_front_right_link" reason="Never"/>
+    <disable_collisions link1="lidar_2_link" link2="mpo_500_wheel_back_left_link" reason="Never"/>
+    <disable_collisions link1="lidar_2_link" link2="mpo_500_wheel_back_right_link" reason="Never"/>
+    <disable_collisions link1="lidar_2_link" link2="mpo_500_wheel_front_left_link" reason="Never"/>
+    <disable_collisions link1="lidar_2_link" link2="mpo_500_wheel_front_right_link" reason="Never"/>
     <disable_collisions link1="lidar_2_link" link2="${prefix_value}base_link_inertia" reason="Never"/>
     <disable_collisions link1="lidar_2_link" link2="${prefix_value}shoulder_link" reason="Never"/>
     <disable_collisions link1="lidar_2_link" link2="${prefix_value}upper_arm_link" reason="Never"/>
-    <disable_collisions link1="mpo_500_omni_wheel_back_left_link" link2="mpo_500_omni_wheel_back_right_link" reason="Never"/>
-    <disable_collisions link1="mpo_500_omni_wheel_back_left_link" link2="mpo_500_omni_wheel_front_left_link" reason="Never"/>
-    <disable_collisions link1="mpo_500_omni_wheel_back_left_link" link2="mpo_500_omni_wheel_front_right_link" reason="Never"/>
-    <disable_collisions link1="mpo_500_omni_wheel_back_left_link" link2="${prefix_value}base_link_inertia" reason="Never"/>
-    <disable_collisions link1="mpo_500_omni_wheel_back_left_link" link2="${prefix_value}shoulder_link" reason="Never"/>
-    <disable_collisions link1="mpo_500_omni_wheel_back_left_link" link2="${prefix_value}upper_arm_link" reason="Never"/>
-    <disable_collisions link1="mpo_500_omni_wheel_back_right_link" link2="mpo_500_omni_wheel_front_left_link" reason="Never"/>
-    <disable_collisions link1="mpo_500_omni_wheel_back_right_link" link2="mpo_500_omni_wheel_front_right_link" reason="Never"/>
-    <disable_collisions link1="mpo_500_omni_wheel_back_right_link" link2="${prefix_value}base_link_inertia" reason="Never"/>
-    <disable_collisions link1="mpo_500_omni_wheel_back_right_link" link2="${prefix_value}shoulder_link" reason="Never"/>
-    <disable_collisions link1="mpo_500_omni_wheel_back_right_link" link2="${prefix_value}upper_arm_link" reason="Never"/>
-    <disable_collisions link1="mpo_500_omni_wheel_front_left_link" link2="mpo_500_omni_wheel_front_right_link" reason="Never"/>
-    <disable_collisions link1="mpo_500_omni_wheel_front_left_link" link2="${prefix_value}base_link_inertia" reason="Never"/>
-    <disable_collisions link1="mpo_500_omni_wheel_front_left_link" link2="${prefix_value}shoulder_link" reason="Never"/>
-    <disable_collisions link1="mpo_500_omni_wheel_front_left_link" link2="${prefix_value}upper_arm_link" reason="Never"/>
-    <disable_collisions link1="mpo_500_omni_wheel_front_right_link" link2="${prefix_value}base_link_inertia" reason="Never"/>
-    <disable_collisions link1="mpo_500_omni_wheel_front_right_link" link2="${prefix_value}shoulder_link" reason="Never"/>
-    <disable_collisions link1="mpo_500_omni_wheel_front_right_link" link2="${prefix_value}upper_arm_link" reason="Never"/>
+    <disable_collisions link1="mpo_500_wheel_back_left_link" link2="mpo_500_wheel_back_right_link" reason="Never"/>
+    <disable_collisions link1="mpo_500_wheel_back_left_link" link2="mpo_500_wheel_front_left_link" reason="Never"/>
+    <disable_collisions link1="mpo_500_wheel_back_left_link" link2="mpo_500_wheel_front_right_link" reason="Never"/>
+    <disable_collisions link1="mpo_500_wheel_back_left_link" link2="${prefix_value}base_link_inertia" reason="Never"/>
+    <disable_collisions link1="mpo_500_wheel_back_left_link" link2="${prefix_value}shoulder_link" reason="Never"/>
+    <disable_collisions link1="mpo_500_wheel_back_left_link" link2="${prefix_value}upper_arm_link" reason="Never"/>
+    <disable_collisions link1="mpo_500_wheel_back_right_link" link2="mpo_500_wheel_front_left_link" reason="Never"/>
+    <disable_collisions link1="mpo_500_wheel_back_right_link" link2="mpo_500_wheel_front_right_link" reason="Never"/>
+    <disable_collisions link1="mpo_500_wheel_back_right_link" link2="${prefix_value}base_link_inertia" reason="Never"/>
+    <disable_collisions link1="mpo_500_wheel_back_right_link" link2="${prefix_value}shoulder_link" reason="Never"/>
+    <disable_collisions link1="mpo_500_wheel_back_right_link" link2="${prefix_value}upper_arm_link" reason="Never"/>
+    <disable_collisions link1="mpo_500_wheel_front_left_link" link2="mpo_500_wheel_front_right_link" reason="Never"/>
+    <disable_collisions link1="mpo_500_wheel_front_left_link" link2="${prefix_value}base_link_inertia" reason="Never"/>
+    <disable_collisions link1="mpo_500_wheel_front_left_link" link2="${prefix_value}shoulder_link" reason="Never"/>
+    <disable_collisions link1="mpo_500_wheel_front_left_link" link2="${prefix_value}upper_arm_link" reason="Never"/>
+    <disable_collisions link1="mpo_500_wheel_front_right_link" link2="${prefix_value}base_link_inertia" reason="Never"/>
+    <disable_collisions link1="mpo_500_wheel_front_right_link" link2="${prefix_value}shoulder_link" reason="Never"/>
+    <disable_collisions link1="mpo_500_wheel_front_right_link" link2="${prefix_value}upper_arm_link" reason="Never"/>
     <disable_collisions link1="${prefix_value}base_link_inertia" link2="${prefix_value}shoulder_link" reason="Adjacent"/>
     <disable_collisions link1="${prefix_value}base_link_inertia" link2="${prefix_value}upper_arm_link" reason="Never"/>
@@ -99,3 +101,18 @@
     <disable_collisions link1="${prefix_value}wrist_1_link" link2="${prefix_value}wrist_3_link" reason="Never"/>
     <disable_collisions link1="${prefix_value}wrist_2_link" link2="${prefix_value}wrist_3_link" reason="Adjacent"/>
+    <!-- Gripper Conditions -->
+    <xacro:unless value="${gripper == ''}">
+      <xacro:if value="${gripper == '2f_140'}">
+        <xacro:include filename="$(find neo_ur_moveit_config)/srdf/robotiq_2f_140.srdf.xacro" />
+        <xacro:robotiq_2f_140 />
+      </xacro:if>
+      <xacro:if value="${gripper == '2f_85'}">
+        <xacro:include filename="$(find neo_ur_moveit_config)/srdf/robotiq_2f_85.srdf.xacro" />
+        <xacro:robotiq_2f_85 />
+      </xacro:if>
+      <xacro:if value="${gripper == 'epick'}">
+        <xacro:include filename="$(find neo_ur_moveit_config)/srdf/robotiq_epick.xacro" />
+        <xacro:robotiq_epick />
+      </xacro:if>
+    </xacro:unless>
 </robot>

File: neo_ur_moveit_config/srdf/mpo_700.srdf.xacro (robot description, xacro)
@@ -145,9 +145,13 @@
     <disable_collisions link1="${prefix_value}wrist_1_link" link2="${prefix_value}wrist_3_link" reason="Never"/>
     <disable_collisions link1="${prefix_value}wrist_2_link" link2="${prefix_value}wrist_3_link" reason="Adjacent"/>
-    <!-- Assigning Xacro properties -->
+    <!-- Gripper Conditions -->
     <xacro:unless value="${gripper == ''}">
       <xacro:if value="${gripper == '2f_140'}">
-        <xacro:include filename="$(find neo_ur_moveit_config)/srdf/robotiq_2f_140.xacro" />
+        <xacro:include filename="$(find neo_ur_moveit_config)/srdf/robotiq_2f_140.srdf.xacro" />
         <xacro:robotiq_2f_140 />
+      </xacro:if>
+      <xacro:if value="${gripper == '2f_85'}">
+        <xacro:include filename="$(find neo_ur_moveit_config)/srdf/robotiq_2f_85.srdf.xacro" />
+        <xacro:robotiq_2f_85 />
       </xacro:if>
       <xacro:if value="${gripper == 'epick'}">

File: neo_ur_moveit_config/srdf/robotiq_2f_140.srdf.xacro (robot description, xacro)
@@ -5,21 +5,8 @@
 -->
 <robot xmlns:xacro="http://www.ros.org/wiki/xacro" name="mpo_700">
+  <xacro:arg name="prefix" default=""/>
+  <xacro:property name="prefix_value" value="$(arg prefix)"/>
   <xacro:macro name="robotiq_2f_140">
-    <!--PASSIVE JOINT: Purpose: this element is used to mark joints that are not actuated-->
-    <group name="gripper">
-      <joint name="finger_joint"/>
-    </group>
-    <passive_joint name="right_inner_finger_joint"/>
-    <passive_joint name="right_outer_knuckle_joint"/>
-    <passive_joint name="right_inner_knuckle_joint"/>
-    <passive_joint name="left_inner_knuckle_joint"/>
-    <passive_joint name="left_inner_finger_joint"/>
-    <group_state name="open" group="gripper">
-      <joint name="finger_joint" value="0.0" />
-    </group_state>
-    <group_state name="close" group="gripper">
-      <joint name="finger_joint" value="0.7" />
-    </group_state>
-    <end_effector name="endeffector" parent_link="${prefix_value}wrist_3_link" group="gripper"/>
+    <!--DISABLE COLLISIONS: By default it is assumed that any link of the robot could potentially come into collision with any other link in the robot. This tag disables collision checking between a specified pair of links. -->
     <disable_collisions link1="left_inner_finger" link2="ur_to_robotiq_link" reason="Never"/>
     <disable_collisions link1="left_inner_finger_pad" link2="ur_to_robotiq_link" reason="Never"/>
